Commit message: chore: Update EasyCAT configuration for joint 7

File: description/ros2_control/easycat.ros2_control.xacro (robot description, xacro)
@@ -86,4 +86,17 @@
         </ec_module>
       </joint>
+      <joint name="joint_7">
+        <state_interface name="position"/>
+        <state_interface name="velocity"/>
+        <state_interface name="effort" />
+        <command_interface name="position"/>
+        <ec_module name="easycat">
+          <plugin>ethercat_generic_plugins/EcCiA402Drive</plugin>
+          <param name="alias">0</param>
+          <param name="position">0</param>
+          <param name="mode_of_operation">9</param>
+          <param name="slave_config">$(find ethercat_easycat)/config/easycat_config_joint_7.yaml</param>
+        </ec_module>
+      </joint>
     </ros2_control>
   </xacro:macro>

File: description/ros2_control/easycat_torque.ros2_control.xacro (robot description, xacro)
@@ -86,4 +86,17 @@
         </ec_module>
       </joint>
+      <joint name="joint_7">
+        <state_interface name="position"/>
+        <state_interface name="velocity"/>
+        <state_interface name="effort"/>
+        <command_interface name="effort"/>
+        <ec_module name="easycat">
+          <plugin>ethercat_generic_plugins/EcCiA402Drive</plugin>
+          <param name="alias">0</param>
+          <param name="position">0</param>
+          <param name="mode_of_operation">9</param>
+          <param name="slave_config">$(find ethercat_easycat)/config/easycat_config_joint_7_torque.yaml</param>
+        </ec_module>
+      </joint>
     </ros2_control>
   </xacro:macro>

File: description/ros2_control/easycat_velocity.ros2_control.xacro (robot description, xacro)
@@ -86,4 +86,17 @@
         </ec_module>
       </joint>
+      <joint name="joint_7">
+        <state_interface name="position"/>
+        <state_interface name="velocity"/>
+        <state_interface name="effort"/>
+        <command_interface name="velocity"/>
+        <ec_module name="easycat">
+          <plugin>ethercat_generic_plugins/EcCiA402Drive</plugin>
+          <param name="alias">0</param>
+          <param name="position">0</param>
+          <param name="mode_of_operation">9</param>
+          <param name="slave_config">$(find ethercat_easycat)/config/easycat_config_joint_7_velocity.yaml</param>
+        </ec_module>
+      </joint>
     </ros2_control>
   </xacro:macro>
